Commit message: changed assets

File: nuro_arm/assets/urdf/xarm.urdf (robot description, URDF)
Before this commit: robot xarm, 13 links, 12 joints
Links:
- added link camera_link, mass 0.001; visual box size=0.008 0.012 0.005
- link base_link: geometry collision box size=0.07606218 0.0770 0.0320; collision box size=0.15400229 0.1400 0.0020
- link forearm_link: geometry collision box size=0.023 0.035 0.09; visual mesh filename=assets/meshes/forearm.stl scale=0.001 0.001 0.001
- link hand_link: geometry collision box size=0.03 0.04 0.02; collision cylinder length=0.00451872 radius=0.025
- link left_finger_base_link: geometry collision box size=0.003 0.01 0.0375; visual mesh filename=assets/meshes/finger_base.stl scale=0.001 0.001 0.001
- link left_finger_tip_link: geometry collision box size=0.008 0.008 0.012; visual mesh filename=assets/meshes/finger_tip.stl scale=0.001 0.001 0.001
- link right_finger_base_link: geometry collision box size=0.003 0.01 0.0375; visual mesh filename=assets/meshes/finger_base.stl scale=0.001 0.001 0.001
- link right_finger_tip_link: geometry collision box size=0.008 0.008 0.012; visual mesh filename=assets/meshes/finger_tip.stl scale=0.001 0.001 0.001
- link swivel_link: geometry collision box size=0.04350001 0.0400 0.02775; visual mesh filename=assets/meshes/swivel.stl scale=0.001 0.001 0.001
- link upperarm_link: geometry collision box size=0.032 0.056 0.11; visual mesh filename=assets/meshes/upperarm.stl scale=0.001 0.001 0.001
- link wrist_link: geometry collision box size=0.045 0.047 0.06475; visual mesh filename=assets/meshes/wrist.stl scale=0.001 0.001 0.001
Joints:
- added joint camera_joint: type fixed, parent hand_link, child camera_link, origin xyz=-0.025 0.0 0.05 rpy=0 0 0

Commit message: latest

File: nuro_arm/assets/urdf/xarm.urdf (robot description, URDF)
Before this commit: robot xarm, 14 links, 13 joints
Joints:
- joint camera_joint: origin xyz=-0.025 0.0 0.05 rpy=0 0 0 -> xyz=-0.025 0.0 0.03 rpy=0 3.14159 1.5708
